Commit message: Update:新增尾部摆动脚本，正常加载机器鱼到水下环境

File: src/shark_test_description/robots/default.xacro (robot description, xacro)
@@ -3,29 +3,23 @@
   <xacro:arg name="debug" default="0"/>
   <xacro:arg name="namespace" default="shark_test"/>
-  <!-- Include the ROV macro file -->
+  <xacro:arg name="inertial_reference_frame" default="world"/>
   <xacro:include filename="$(find shark_test_description)/urdf/base.xacro"/>
-  <xacro:include filename="$(find shark_test_description)/urdf/gazebo.xacro"/>
-  <!-- Create the shark_test -->
-  <xacro:shark_test_base namespace="$(arg namespace)">
-    <!-- The underwater object plugin is given as an input block parameter to
-     allow the addition of external models of manipulator units -->
+  <!-- 创建机器鱼基础模型 -->
+  <xacro:shark_test_base
+    namespace="$(arg namespace)"
+    inertial_reference_frame="$(arg inertial_reference_frame)">
+        <!-- 水下物体插件 -->
     <gazebo>
       <plugin name="uuv_plugin" filename="libuuv_underwater_object_ros_plugin.so">
+        <link_name>$(arg namespace)/base_link</link_name>  <!-- 使用命名空间变量 -->
         <fluid_density>1028.0</fluid_density>
-        <flow_velocity_topic>hydrodynamics/current_velocity</flow_velocity_topic>
-        <debug>$(arg debug)</debug>
-        <!-- Adding the hydrodynamic and hydrostatic parameters for the vehicle-->
-        <xacro:shark_test_hydro_model namespace="$(arg namespace)"/>
-        <!--
-          In case other modules are added to the vehicle (such as a manipulator)
-          that also have link running with the underwater object plugin, they
-          should also be added in this block. For this, this new module should
-          have a file similar to gazebo.xacro above with the description of the
-          parameter necessary for the underwater object plugin to be initialized.
-        -->
+        <flow_velocity_topic>/hydrodynamics/current_velocity</flow_velocity_topic>
+        <debug>true</debug>
+        <use_global_current>true</use_global_current>
+        <enable_buoyancy_debug>true</enable_buoyancy_debug>
       </plugin>
     </gazebo>
   </xacro:shark_test_base>
-  <!-- Joint state publisher plugin -->
-  <xacro:default_joint_state_publisher namespace="$(arg namespace)" update_rate="10"/>
+  <!-- 关节状态发布器 -->
+  <xacro:default_joint_state_publisher namespace="$(arg namespace)" update_rate="20"/>
 </robot>

File: src/shark_test_description/urdf/actuators.xacro (robot description, xacro)
@@ -1,49 +1,74 @@
 <?xml version="1.0"?>
 <robot xmlns:xacro="http://www.ros.org/wiki/xacro">
-    <!-- Adding the fin units with the macro created in snippets.xacro -->
-    <!--
-    Important:
-        - The fin IDs must be given as integers and must be unique to each fin unit
-        - The fin pose in the <origin> block is relative to the parent link's origin
-    -->
-    <!-- 胸鳍（父连杆：base_link） -->
-    <xacro:fin_macro
-        namespace="${namespace}"
-        fin_id="0"
-        parent_link="${namespace}/base_link"
-        mesh_file="package://shark_test_description/meshes/body_fin.stl">
-        <origin xyz="0.0 0 0" rpy="0 0 0" />  <!-- 胸鳍在base_link前方0.05米 -->
-    </xacro:fin_macro>
-    <!-- 尾鳍link1（父连杆：base_link） -->
-    <xacro:fin_macro
-        namespace="${namespace}"
-        fin_id="1"
-        parent_link="${namespace}/base_link"
-        mesh_file="package://shark_test_description/meshes/link1.stl">
-        <origin xyz="0.169 0 0" rpy="0 0 0" />  <!-- link1在base_link后方0.169米 -->
-    </xacro:fin_macro>
-    <!-- 尾鳍link2（父连杆：fin1） -->
-    <xacro:fin_macro
-        namespace="${namespace}"
-        fin_id="2"
-        parent_link="${namespace}/fin1"
-        mesh_file="package://shark_test_description/meshes/link2.stl">
-        <origin xyz="0.062 0 0" rpy="0 0 0" />  <!-- link2在link1末端（x=0.062米） -->
-    </xacro:fin_macro>
-    <!-- 尾鳍link3（父连杆：fin2） -->
-    <xacro:fin_macro
-        namespace="${namespace}"
-        fin_id="3"
-        parent_link="${namespace}/fin2"
-        mesh_file="package://shark_test_description/meshes/link3.stl">
-        <origin xyz="0.062 0 0" rpy="0 0 0" />
-    </xacro:fin_macro>
-    <!-- 尾鳍link4（父连杆：fin3） -->
-    <xacro:fin_macro
-        namespace="${namespace}"
-        fin_id="4"
-        parent_link="${namespace}/fin3"
-        mesh_file="package://shark_test_description/meshes/link4.stl">
-        <origin xyz="0.064 0 0" rpy="0 0 0" />
-    </xacro:fin_macro>
+  <!-- 基于base.xacro的位置参数，配置5个鱼鳍（修复胸鳍关节锁死） -->
+  <!-- 1. 胸鳍（fin0）：修正effort和velocity，避免锁死 -->
+  <xacro:fin_macro
+      namespace="${namespace}"
+      fin_id="0"
+      parent_link="${namespace}/base_link"
+      mesh_file="package://shark_test_description/meshes/body_fin.STL"
+      lower_limit="-0.52"
+      upper_limit="0.52"
+      effort="5.0"
+      velocity="2.0"
+      axis="0 1 0"
+      mass="0.78" >  <!-- 绕y轴转动（上下摆动） -->
+      <origin xyz="0 0 0" rpy="0 0 0" />
+  </xacro:fin_macro>
+  <!-- 2. 尾鳍link1（fin1）：保留原有参数 -->
+  <xacro:fin_macro
+      namespace="${namespace}"
+      fin_id="1"
+      parent_link="${namespace}/base_link"
+      mesh_file="package://shark_test_description/meshes/link1.STL"
+      lower_limit="-0.54777"
+      upper_limit="0.54777"
+      effort="5.0"
+      velocity="2.0"
+      axis="0 0 1"
+      mass="0.28">  <!-- 绕z轴转动（左右摆动） -->
+      <origin xyz="0.16952 -0.001 0.022" rpy="0 0 0" />
+  </xacro:fin_macro>
+  <!-- 3. 尾鳍link2（fin2）：保留原有参数 -->
+  <xacro:fin_macro
+      namespace="${namespace}"
+      fin_id="2"
+      parent_link="${namespace}/fin1"
+      mesh_file="package://shark_test_description/meshes/link2.STL"
+      lower_limit="-0.5242"
+      upper_limit="0.5242"
+      effort="5.0"
+      velocity="2.0"
+      axis="0 0 -1"
+      mass="0.23" >  <!-- 绕z轴反向转动 -->
+      <origin xyz="0.06502 0 0" rpy="0 0 0" />
+  </xacro:fin_macro>
+  <!-- 4. 尾鳍link3（fin3）：保留原有参数 -->
+  <xacro:fin_macro
+      namespace="${namespace}"
+      fin_id="3"
+      parent_link="${namespace}/fin2"
+      mesh_file="package://shark_test_description/meshes/link3.STL"
+      lower_limit="-0.424"
+      upper_limit="0.424"
+      effort="4.0"
+      velocity="1.5"
+      axis="0 0 1"
+      mass="0.19" >
+      <origin xyz="0.06402 0 0" rpy="0 0 0" />
+  </xacro:fin_macro>
+  <!-- 5. 尾鳍link4（fin4）：保留原有参数 -->
+  <xacro:fin_macro
+      namespace="${namespace}"
+      fin_id="4"
+      parent_link="${namespace}/fin3"
+      mesh_file="package://shark_test_description/meshes/link4.STL"
+      lower_limit="-0.265"
+      upper_limit="0.265"
+      effort="2.0"
+      velocity="1.0"
+      axis="0 0 -1"
+      mass="0.11" >
+      <origin xyz="0.0668 0 0" rpy="0 0 0" />
+  </xacro:fin_macro>
 </robot>

File: src/shark_test_description/urdf/base.xacro (robot description, xacro)
@@ -1,36 +1,28 @@
 <?xml version="1.0"?>
 <robot xmlns:xacro="http://www.ros.org/wiki/xacro">
-  <!-- Loading some constants -->
+  <!-- 引入依赖宏文件 -->
   <xacro:include filename="$(find uuv_descriptions)/urdf/common.urdf.xacro"/>
-  <!-- Loading file with sensor macros -->
   <xacro:include filename="$(find uuv_sensor_ros_plugins)/urdf/sensor_snippets.xacro"/>
-  <!-- Loading the UUV simulator ROS plugin macros -->
   <xacro:include filename="$(find uuv_gazebo_ros_plugins)/urdf/snippets.xacro"/>
-  <!-- Loading vehicle's specific macros -->
   <xacro:include filename="$(find shark_test_description)/urdf/snippets.xacro"/>
-  <!--
-    Vehicle's parameters (remember to enter the model parameters below)
-  -->
-  <xacro:property name="mass" value="3.473"/>
-  <!-- Center of gravity -->
+  <!-- 机器鱼核心参数（包含水动力参数） -->
+  <xacro:property name="mass" value="0.003"/>  <!--1.753-->
   <xacro:property name="cog" value="0.038191 -0.0011682 0.019734"/>
-  <!-- Fluid density -->
+  <xacro:property name="cob" value="0.038191 -0.0011682 0.029734"/>  <!-- 浮心 -->
+  <xacro:property name="volume" value="0.004"/>  <!-- 排水体积 -->
   <xacro:property name="rho" value="1028"/>
-  <!-- 网格文件路径 -->
   <xacro:property name="base_link_mesh" value="package://shark_test_description/meshes/base_link.STL"/>
-  <xacro:property name="body_fin_mesh" value="package://shark_test_description/meshes/body_fin.STL"/>
-  <xacro:property name="link1_mesh" value="package://shark_test_description/meshes/link1.STL"/>
-  <xacro:property name="link2_mesh" value="package://shark_test_description/meshes/link2.STL"/>
-  <xacro:property name="link3_mesh" value="package://shark_test_description/meshes/link3.STL"/>
-  <xacro:property name="link4_mesh" value="package://shark_test_description/meshes/link4.STL"/>
-  <xacro:macro name="shark_test_base" params="namespace *gazebo">
-    <!-- 1. 基础连杆 base_link（复用原有惯性、可视化、碰撞） -->
+  <!-- 机器鱼基础模型宏 -->
+  <xacro:macro name="shark_test_base" params="namespace *gazebo inertial_reference_frame">
+    <!-- 核心连杆base_link（整合水动力参数） -->
     <link name="${namespace}/base_link">
+      <!-- 惯性参数 -->
       <inertial>
-        <mass value="1.753" />
-        <origin xyz="0.038191 -0.0011682 0.019734" rpy="0 0 0"/>
+        <mass value="${mass}" />
+        <origin xyz="${cog}" rpy="0 0 0"/>
         <inertia ixx="0.0011992" ixy="-5.9532E-07" ixz="-4.094E-05"
                  iyy="0.0049871" iyz="-7.025E-07" izz="0.0055025" />
       </inertial>
+      <!-- 可视化模型 -->
       <visual>
         <origin xyz="0 0 0" rpy="0 0 0"/>
@@ -40,4 +32,5 @@
         <material name="white"><color rgba="1 1 1 1" /></material>
       </visual>
+      <!-- 碰撞体 -->
       <collision>
         <origin xyz="0 0 0" rpy="0 0 0"/>
@@ -46,179 +39,43 @@
         </geometry>
       </collision>
-    </link>
-    <!-- 2. 胸鳍连杆 body_fin -->
-    <link name="${namespace}/body_fin">
-      <inertial>
-        <mass value="0.0777166528344648" />
-        <origin xyz="0.00914833180910446 -0.00106620065635634 2.43483887424727E-05" rpy="0 0 0"/>
-        <inertia ixx="3.1049811920015E-05" ixy="-3.79774234954185E-10" ixz="-3.71777530984048E-08"
-                 iyy="1.59640204823738E-05" iyz="1.84244309068481E-07" izz="4.63071029422297E-05" />
-      </inertial>
-      <visual>
-        <origin xyz="0 0 0" rpy="0 0 0"/>
+      <collision>
+        <origin xyz="${cog}" rpy="0 0 0"/>
         <geometry>
-          <mesh filename="${body_fin_mesh}" scale="1 1 1" />
-        </geometry>
-        <material name="light_gray"><color rgba="0.898 0.918 0.929 1" /></material>
-      </visual>
-      <collision>
-        <origin xyz="0 0 0" rpy="0 0 0"/>
-        <geometry>
-          <mesh filename="${body_fin_mesh}" scale="1 1 1" />
+          <box size="0.65 0.32 0.25"/>
         </geometry>
       </collision>
+      <!-- 关键：直接在base_link内添加水动力参数 -->
+      <neutrally_buoyant>0</neutrally_buoyant>
+      <volume>${volume}</volume>
+      <center_of_buoyancy>${cob}</center_of_buoyancy>
+      <box>
+        <width>0.32</width>
+        <length>0.65</length>
+        <height>0.25</height>
+      </box>
+      <hydrodynamic_model>
+        <type>fossen</type>
+        <added_mass>
+          0.1   0      0      0      0      0
+          0    0.08    0      0      0      0
+          0     0     0.12    0      0      0
+          0     0      0     0.01    0      0
+          0     0      0      0     0.01    0
+          0     0      0      0      0     0.01
+        </added_mass>
+        <linear_damping>200 150 150 50 50 50</linear_damping>  <!-- 增大20倍 -->
+        <quadratic_damping>1000 800 800 300 300 300</quadratic_damping>
+      </hydrodynamic_model>
     </link>
-    <!-- 胸鳍关节 body_fin_joint -->
-    <joint name="${namespace}/body_fin_joint" type="revolute">
-      <origin xyz="0 0 0" rpy="0 0 0" />
-      <parent link="${namespace}/base_link" />
-      <child link="${namespace}/body_fin" />
-      <axis xyz="0 1 0" />
-      <limit lower="-0.52" upper="0.52" effort="0" velocity="0" />
-    </joint>
-    <!-- 3. 尾鳍连杆 link1 -->
-    <link name="${namespace}/link1">
-      <inertial>
-        <mass value="0.276636032216536" />
-        <origin xyz="0.0273740098565554 1.00730841318137E-06 0.00233674443466103" rpy="0 0 0"/>
-        <inertia ixx="0.000221100847637612" ixy="2.2348802662522E-08" ixz="1.48015173973935E-06"
-                 iyy="0.000306819552826337" iyz="-1.51964922899048E-08" izz="0.000127523807633018" />
-      </inertial>
-      <visual>
-        <origin xyz="0 0 0" rpy="0 0 0"/>
-        <geometry>
-          <mesh filename="${link1_mesh}" scale="1 1 1" />
-        </geometry>
-        <material name="white"><color rgba="1 1 1 1" /></material>
-      </visual>
-      <collision>
-        <origin xyz="0 0 0" rpy="0 0 0"/>
-        <geometry>
-          <mesh filename="${link1_mesh}" scale="1 1 1" />
-        </geometry>
-      </collision>
-    </link>
-    <!-- 尾鳍关节 joint1 -->
-    <joint name="${namespace}/joint1" type="revolute">
-      <origin xyz="0.16952 -0.001 0.022" rpy="0 0 0" />
-      <parent link="${namespace}/base_link" />
-      <child link="${namespace}/link1" />
-      <axis xyz="0 0 1" />
-      <limit lower="-0.54777" upper="0.54777" effort="5.0" velocity="2.0" />
-    </joint>
-    <!-- 4. 尾鳍连杆 link2 -->
-    <link name="${namespace}/link2">
-      <inertial>
-        <mass value="0.23079291425153" />
-        <origin xyz="0.0314265398767537 7.62073086331302E-06 0.00321188485864419" rpy="0 0 0"/>
-        <inertia ixx="0.00014162458840055" ixy="1.43555615633064E-07" ixz="6.00764632389094E-06"
-                 iyy="0.000192380669161936" iyz="7.81445755193396E-09" izz="0.000124286520292589" />
-      </inertial>
-      <visual>
-        <origin xyz="0 0 0" rpy="0 0 0"/>
-        <geometry>
-          <mesh filename="${link2_mesh}" scale="1 1 1" />
-        </geometry>
-        <material name="white"><color rgba="1 1 1 1" /></material>
-      </visual>
-      <collision>
-        <origin xyz="0 0 0" rpy="0 0 0"/>
-        <geometry>
-          <mesh filename="${link2_mesh}" scale="1 1 1" />
-        </geometry>
-      </collision>
-    </link>
-    <!-- 尾鳍关节 joint2 -->
-    <joint name="${namespace}/joint2" type="revolute">
-      <origin xyz="0.06502 0 0" rpy="0 0 0" />
-      <parent link="${namespace}/link1" />
-      <child link="${namespace}/link2" />
-      <axis xyz="0 0 -1" />
-      <limit lower="-0.5242" upper="0.5242" effort="5.0" velocity="2.0" />
-    </joint>
-    <!-- 5. 尾鳍连杆 link3 -->
-    <link name="${namespace}/link3">
-      <inertial>
-        <mass value="0.194723948866163" />
-        <origin xyz="0.0326080633640175 0.000105371441976573 0.00539746824234997" rpy="0 0 0"/>
-        <inertia ixx="7.98162926930531E-05" ixy="-2.49207714784249E-07" ixz="4.9950223786246E-06"
-                 iyy="0.00012964160787792" iyz="7.02465415687571E-09" izz="9.38054135694122E-05" />
-      </inertial>
-      <visual>
-        <origin xyz="0 0 0" rpy="0 0 0"/>
-        <geometry>
-          <mesh filename="${link3_mesh}" scale="1 1 1" />
-        </geometry>
-        <material name="light_gray"><color rgba="0.898 0.918 0.929 1" /></material>
-      </visual>
-      <collision>
-        <origin xyz="0 0 0" rpy="0 0 0"/>
-        <geometry>
-          <mesh filename="${link3_mesh}" scale="1 1 1" />
-        </geometry>
-      </collision>
-    </link>
-    <!-- 尾鳍关节 joint3 -->
-    <joint name="${namespace}/joint3" type="revolute">
-      <origin xyz="0.06402 0 0" rpy="0 0 0" />
-      <parent link="${namespace}/link2" />
-      <child link="${namespace}/link3" />
-      <axis xyz="0 0 1" />
-      <limit lower="-0.424" upper="0.424" effort="4.0" velocity="1.5" />
-    </joint>
-    <!-- 6. 尾鳍连杆 link4 -->
-    <!-- 尾巴连杆4（尾鳍，用 link4.stl） -->
-    <link name="${namespace}/link4">
-      <inertial>
-        <mass value="0.005"/> <!-- 尾鳍质量略大于其他尾柄连杆 -->
-        <origin xyz="0 0 0" rpy="0 0 0"/>
-        <inertia ixx="5e-6" ixy="0" ixz="0" iyy="5e-6" iyz="0" izz="2e-6"/>
-      </inertial>
-      <!-- 可视化：替换为 link4.stl（和鳍宏的尾鳍区分开？或统一用一个？） -->
-      <!-- 注意：如果你的尾鳍是“尾巴最后一个连杆”，而非独立鳍，这里直接用 STL；如果是独立鳍，保持之前的鳍宏配置即可 -->
-      <visual>
-        <origin xyz="0 0 0" rpy="0 0 0"/>
-        <geometry>
-          <mesh filename="package://shark_test_description/meshes/link4.STL" scale="1 1 1"/>
-        </geometry>
-        <material name="blue"><color rgba="0 0 1 1"/></material>
-      </visual>
-      <collision>
-        <origin xyz="0 0 0" rpy="0 0 0"/>
-        <geometry><box size="0.04 0.05 0.02"/></geometry> <!-- 碰撞简化，适配 STL 尺寸 -->
-      </collision>
-    </link>
-    <!-- joint4 -->
-    <joint name="${namespace}/joint4" type="revolute">
-      <origin xyz="0.0668 0 0" rpy="0 0 0" />
-      <parent link="${namespace}/link3" />
-      <child link="${namespace}/link4" />
-      <axis xyz="0 0 -1" />
-      <limit lower="-0.265" upper="0.265" effort="2.0" velocity="1.0" />
-    </joint>
-    <!-- Gazebo 自碰撞设置 -->
+    <!-- Gazebo自碰撞设置 -->
     <gazebo reference="${namespace}/base_link">
       <selfCollide>false</selfCollide>
+      <max_contacts>10</max_contacts>
     </gazebo>
-    <gazebo reference="${namespace}/body_fin">
-      <selfCollide>false</selfCollide>
-    </gazebo>
-    <gazebo reference="${namespace}/link1">
-      <selfCollide>false</selfCollide>
-    </gazebo>
-    <gazebo reference="${namespace}/link2">
-      <selfCollide>false</selfCollide>
-    </gazebo>
-    <gazebo reference="${namespace}/link3">
-      <selfCollide>false</selfCollide>
-    </gazebo>
-    <gazebo reference="${namespace}/link4">
-      <selfCollide>false</selfCollide>
-    </gazebo>
-    <!-- 插入流体动力学插件 -->
+    <!-- 插入gazebo插件块 -->
     <xacro:insert_block name="gazebo"/>
-    <!-- 包含执行器（推进器、鳍）和传感器 -->
+    <!-- 包含执行器和传感器 -->
     <xacro:include filename="$(find shark_test_description)/urdf/actuators.xacro"/>
     <xacro:include filename="$(find shark_test_description)/urdf/sensors.xacro"/>
-    </xacro:macro>
+  </xacro:macro>
 </robot>
