Commit message: Update:新增尾部摆动脚本，正常加载机器鱼到水下环境

File: src/shark_test_description/urdf/gazebo.xacro (robot description, xacro)
@@ -1,97 +1,35 @@
 <?xml version="1.0"?>
 <robot xmlns:xacro="http://www.ros.org/wiki/xacro">
-    <!-- Center of buoyancy -->
-    <xacro:property name="shark_test_cob" value="0.038191 -0.0011682 0.029734"/>
-    <!-- Vehicle's actual volume (Gazebo cannot compute the volume out of the mesh) -->
-    <xacro:property name="shark_test_volume" value="0.0035"/>
-    <!-- Describing the dimensions of the vehicle's bounding box -->
-    <xacro:property name="shark_test_length" value="0.65"/>
-    <xacro:property name="shark_test_width"  value="0.32"/>
-    <xacro:property name="shark_test_height" value="0.25"/>
-    <xacro:macro name="shark_test_hydro_model" params="namespace">
-      <!-- List of hydrodynamic models this robot's links -->
-      <link name="${namespace}/base_link">
-        <!-- This flag will make the link neutrally buoyant -->
+  <!-- 机器鱼水动力核心参数（与base_link尺寸匹配） -->
+  <xacro:property name="shark_test_cob" value="0.038191 -0.0011682 0.029734"/>  <!-- 浮心（z轴高于重心） -->
+  <xacro:property name="shark_test_volume" value="0.04"/>  <!-- 排水体积（浮力≈40N>重力≈34N） -->
+  <xacro:property name="shark_test_length" value="0.65"/>  <!-- 体长 -->
+  <xacro:property name="shark_test_width"  value="0.32"/>  <!-- 体宽 -->
+  <xacro:property name="shark_test_height" value="0.25"/>  <!-- 体高 -->
+  <!-- 水动力模型宏（写入base_link的参数，供插件读取） -->
+  <xacro:macro name="shark_test_hydro_model" params="namespace">
+        <xacro:modify_link name="${namespace}/base_link">
         <neutrally_buoyant>0</neutrally_buoyant>
-        <!-- Link's volume -->
         <volume>${shark_test_volume}</volume>
-        <!-- Link's bounding box, it is used to recalculate the immersed
-        volume when close to the surface.
-        This is a workaround the invalid bounding box given by Gazebo-->
+        <center_of_buoyancy>${shark_test_cob}</center_of_buoyancy>
         <box>
-          <width>${shark_test_width}</width>
-          <length>${shark_test_length}</length>
-          <height>${shark_test_height}</height>
+            <width>${shark_test_width}</width>
+            <length>${shark_test_length}</length>
+            <height>${shark_test_height}</height>
         </box>
-        <!-- Center of buoyancy -->
-        <center_of_buoyancy>${shark_test_cob}</center_of_buoyancy>
-        <!--
-        Choose one of the hydrodynamic models below, all are based on
-        Fossen's equation of motion for underwater vehicles
-        Reference:
-        [1] Fossen, Thor I. Handbook of marine craft hydrodynamics and motion
-            control. John Wiley & Sons, 2011.
-        -->
-        <!-- 1) Fossen's equation of motion -->
         <hydrodynamic_model>
-          <type>fossen</type>
-          <added_mass>
-            0.1 0 0 0 0 0
-            0 0.05 0 0 0 0
-            0 0 0.05 0 0 0
-            0 0 0 0.001 0 0
-            0 0 0 0 0.001 0
-            0 0 0 0 0 0.001
-          </added_mass>
-          <!--
-            The linear damping coefficients can be provided as a diagonal (6 elements)
-            or a full matrix (36 coefficients), like the added-mass coefficients above
-          -->
-          <linear_damping>
-            5 3 3 0.5 0.5 0.5
-          </linear_damping>
-          <!--
-            The linear damping coefficients proportional to the forward speed
-            can be provided as a diagonal (6 elements) or a full matrix (36 coefficients),
-            like the added-mass coefficients above.
-            This matrix is mostly useful for slender bodies (e.g. AUVs with torpedo shape)
-          -->
-          <!-- <linear_damping_forward_speed>
-            0 0 0 0 0 0
-          </linear_damping_forward_speed> -->
-          <!--
-            The quadratic damping coefficients can be provided as a diagonal (6 elements)
-            or a full matrix (36 coefficients), like the added-mass coefficients above
-          -->
-          <quadratic_damping>
-            10 8 8 1 1 1
-          </quadratic_damping>
-          <!--
-            In case you want to model a simple surface vessel, you can use the
-            implementation of linear (small angle) theory for boxed shaped vessels
-            by providing the following parameters. If you omit the area of the
-            water level plane area, it will be calculated from the bounding box
-            parameters. Uncomment the lines below in case you are simulating a
-            surface vessel.
-            For more details on these parameters and the computation of buoyancy
-            for vessels using this theory, check:
-              [1] Lecture Notes  TTK 4190 Guidance and Control of Vehicles (T. I. Fossen)
-                  http://www.fossen.biz/wiley/Ch4.pdf
-              [2] Fossen, Thor I. Handbook of marine craft hydrodynamics and motion
-                  control. John Wiley & Sons, 2011.
-          -->
-          <!--
-          <metacentric_width>0.0</metacentric_width>
-          <metacentric_length>0.0</metacentric_length>
-          <submerged_height>0.0</submerged_height>
-          -->
+            <type>fossen</type>
+            <added_mass>
+            0.1   0      0      0      0      0
+            0    0.08    0      0      0      0
+            0     0     0.12    0      0      0
+            0     0      0     0.01    0      0
+            0     0      0      0     0.01    0
+            0     0      0      0      0     0.01
+            </added_mass>
+            <linear_damping>8 5 5 0.8 0.8 0.8</linear_damping>
+            <quadratic_damping>100 80 80 20 20 20</quadratic_damping>
         </hydrodynamic_model>
-        <!-- 2) This computes the added-mass and damping parameters for a sphere
-        in the fluid with the given radius -->
-        <hydrodynamic_model>
-          <type>sphere</type>
-          <radius>0</radius>
-        </hydrodynamic_model>
-      </link>
-    </xacro:macro>
+        </xacro:modify_link>
+  </xacro:macro>
 </robot>

File: src/shark_test_description/urdf/sensors.xacro (robot description, xacro)
@@ -24,14 +24,14 @@
   </xacro:default_rpt> -->
   <!-- Pressure  -->
-  <xacro:default_pressure namespace="${namespace}" parent_link="${namespace}/base_link">
+  <!-- <xacro:default_pressure namespace="${namespace}" parent_link="${namespace}/base_link">
     <origin xyz="0 0 0" rpy="0 0 0"/>
-  </xacro:default_pressure>
+  </xacro:default_pressure> -->
   <!-- IMU  -->
-  <xacro:default_imu namespace="${namespace}" parent_link="${namespace}/base_link">
+  <!-- <xacro:default_imu namespace="${namespace}" parent_link="${namespace}/base_link">
     <origin xyz="0 0 0" rpy="0 0 0"/>
-  </xacro:default_imu>
+  </xacro:default_imu> -->
   <!-- Mount a camera  -->
-  <xacro:default_camera namespace="${namespace}" parent_link="${namespace}/base_link" suffix="">
+  <!-- <xacro:default_camera namespace="${namespace}" parent_link="${namespace}/base_link" suffix="">
     <origin xyz="0 0 0" rpy="0 0 0"/>
-  </xacro:default_camera>
+  </xacro:default_camera> -->
 </robot>

File: src/shark_test_description/urdf/snippets.xacro (robot description, xacro)
@@ -7,7 +7,7 @@
     fins, you can erase the macro below.
   -->
-  <!-- Fin joint limits  -->
-  <xacro:property name="fin_min_joint_limit" value="${-0.5 * d2r}"/>  <!-- ±28.6度，约±0.5弧度 -->
-  <xacro:property name="fin_max_joint_limit" value="${0.5 * d2r}"/>
+  <!-- 移除硬编码的鳍限位（改为通过参数传递） -->
+  <!-- <xacro:property name="fin_min_joint_limit" value="${-0.5 * d2r}"/> -->
+  <!-- <xacro:property name="fin_max_joint_limit" value="${0.5 * d2r}"/> -->
   <!-- 宏参数说明：
        - namespace: 机器人命名空间
@@ -16,11 +16,16 @@
        - mesh_file: 鳍的网格文件路径（package://格式）
        - *origin: 关节位置/姿态
+       - axis: 关节旋转轴（新增）
+       - lower_limit: 关节下限（新增）
+       - upper_limit: 关节上限（新增）
+       - effort: 关节最大力（新增）
+       - velocity: 关节最大速度（新增）
   -->
-  <xacro:macro name="fin_macro" params="namespace fin_id parent_link:=${namespace}/base_link mesh_file *origin">
+  <xacro:macro name="fin_macro" params="namespace fin_id parent_link:=${namespace}/base_link mesh_file *origin axis lower_limit upper_limit effort velocity mass:=0.03">
       <joint name="${namespace}/fin${fin_id}_joint" type="revolute">
-          <!-- 关节限制：effort和velocity设为非0值，否则关节无法运动 -->
-          <limit effort="50" lower="${fin_min_joint_limit}" upper="${fin_max_joint_limit}" velocity="10"/>
+          <!-- 使用传入的限位、effort、velocity参数 -->
+          <limit effort="${effort}" lower="${lower_limit}" upper="${upper_limit}" velocity="${velocity}"/>
           <xacro:insert_block name="origin"/>
-          <axis xyz="0 0 1"/>  <!-- 绕Z轴旋转（胸鳍左右摆/尾鳍上下摆） -->
+          <axis xyz="${axis}"/>  <!-- 使用传入的旋转轴参数 -->
           <parent link="${parent_link}" />
           <child link="${namespace}/fin${fin_id}" />
@@ -28,5 +33,5 @@
       <link name="${namespace}/fin${fin_id}">
         <inertial>
-          <mass value="0.01" />  <!-- 增大质量，避免Gazebo中模型漂浮 -->
+          <mass value="${mass}" />  <!-- 增大质量，避免Gazebo中模型漂浮 -->
           <origin xyz="0 0 0" rpy="0 0 0"/>
           <inertia ixx="0.0001" ixy="0.0" ixz="0.0"
@@ -50,4 +55,6 @@
       <gazebo>
         <plugin name="${namespace}_fin${fin_id}_model" filename="libuuv_fin_ros_plugin.so">
+          <fin_id>${fin_id}</fin_id>
+          <command_topic>${namespace}/fins/${fin_id}/input</command_topic>
           <!-- 鳍关节动力学模型：一阶延迟，时间常数0.1秒 -->
           <dynamics>
@@ -58,6 +65,8 @@
           <liftdrag>
             <type>Quadratic</type>
-            <lift_constant>10.0</lift_constant>  <!-- 升力系数，需根据鳍尺寸调整 -->
-            <drag_constant>5.0</drag_constant>    <!-- 阻力系数 -->
+            <lift_constant>2000.0</lift_constant>  <!-- 升力系数，越大推力越强 -->
+            <drag_constant>100.0</drag_constant>  <!-- 阻力系数 -->
+            <forward_axis>1 0 0</forward_axis>  <!-- 推力方向（x轴前进） -->
+            <up_axis>0 0 1</up_axis>            <!-- 升力方向（z轴上浮） -->
           </liftdrag>
           <!-- 水动力关键参数 -->
@@ -67,9 +76,8 @@
           <!-- ROS话题配置 -->
           <output_topic>${namespace}/fins/${fin_id}/output</output_topic>
-          <input_topic>${namespace}/fins/${fin_id}/input</input_topic>
           <wrench_topic>${namespace}/fins/${fin_id}/wrench_topic</wrench_topic>
         </plugin>
-        <!-- 新增流体阻力插件，模拟水对鳍的阻尼 -->
-        <plugin name="${namespace}_fin${fin_id}_hydrodynamics" filename="libuuv_hydrodynamic_plugin.so">
+        <!-- 新增流体阻力插件，模拟水对鳍的阻尼（可选启用） -->
+        <!-- <plugin name="${namespace}_fin${fin_id}_hydrodynamics" filename="libuuv_hydrodynamic_plugin.so">
           <link_name>${namespace}/fin${fin_id}</link_name>
           <fluid_density>1000</fluid_density>
@@ -84,5 +92,5 @@
             <z>1.0</z>
           </linear_damping>
-        </plugin>
+        </plugin> -->
       </gazebo>
   </xacro:macro>
